Commit message: Create description files for kinova with rokubi ft sensor

File: kinova_description/urdf/j2n6s300_with_ft.xacro (robot description, xacro)
@@ -16,4 +16,5 @@
     <xacro:include filename="$(find kinova_description)/urdf/kinova_common.xacro" />
     <xacro:include filename="$(find kinova_description)/urdf/kinova_finger_set.xacro" />
+    <xacro:include filename="$(find rokubi_kinova_adapter)/urdf/BFT_ROKS_KINOVA.urdf.xacro" />
     <!-- Import all Gazebo-customization elements -->
     <xacro:include filename="$(find kinova_description)/urdf/kinova.gazebo" />
@@ -108,6 +109,14 @@
         <xacro:kinova_armlink link_name="${prefix}_link_5" link_mesh="${link_5_mesh}" use_ring_mesh="true" ring_mesh="ring_small" mesh_no="${link_5_mesh_no}"/>
         <xacro:kinova_armjoint joint_name="${prefix}_joint_5" type="${joint_5_type}" parent="${prefix}_link_4" child="${prefix}_link_5" joint_axis_xyz="${joint_5_axis_xyz}" joint_origin_xyz="${joint_5_origin_xyz}" joint_origin_rpy="${joint_5_origin_rpy}" joint_velocity_limit="${joint_5_velocity_limit}" joint_torque_limit="${joint_5_torque_limit}"/>
+        <xacro:kinova_virtual_link link_name="${prefix}_ft_robot_side_connector"/>
+        <xacro:kinova_armjoint joint_name="${prefix}_joint_6" type="${joint_6_type}" parent="${prefix}_link_5" child="${prefix}_ft_robot_side_connector" joint_axis_xyz="${joint_6_axis_xyz}" joint_origin_xyz="${joint_6_origin_xyz}" joint_origin_rpy="${joint_6_origin_rpy}" joint_velocity_limit="${joint_6_velocity_limit}" joint_torque_limit="${joint_6_torque_limit}"/>
+        <xacro:BFT_ROKS_KINOVA prefix="${prefix}" />
+        <xacro:kinova_virtual_joint joint_name="${prefix}_joint_ft_robot_side_connector" type="fixed" parent="${prefix}_ft_robot_side_connector" child="${prefix}_robot_side" joint_axis_xyz="0 0 0" joint_origin_xyz="0 0 0" joint_origin_rpy="${J_PI} 0 ${J_PI}" joint_lower_limit="0" joint_upper_limit="0"/>
         <xacro:kinova_armlink link_name="${prefix}_link_6" link_mesh="${link_6_mesh}" use_ring_mesh="true" ring_mesh="ring_small" mesh_no="${link_6_mesh_no}"/>
-        <xacro:kinova_armjoint joint_name="${prefix}_joint_6" type="${joint_6_type}" parent="${prefix}_link_5" child="${prefix}_link_6" joint_axis_xyz="${joint_6_axis_xyz}" joint_origin_xyz="${joint_6_origin_xyz}" joint_origin_rpy="${joint_6_origin_rpy}" joint_velocity_limit="${joint_6_velocity_limit}" joint_torque_limit="${joint_6_torque_limit}"/>
+        <joint name="${prefix}_joint_ft_adapter_to_link_6" type="fixed">
+            <parent link="${prefix}_gripper_adapter" />
+            <child link = "${prefix}_link_6" />
+            <origin xyz="0.0 0.0 0.0" rpy="${J_PI} 0 ${J_PI}" />
+        </joint>
         <xacro:kinova_virtual_link link_name="${prefix}_end_effector"/>
         <xacro:kinova_virtual_joint joint_name="${prefix}_joint_end_effector" type="${joint_end_effector_type}" parent="${prefix}_link_6" child="${prefix}_end_effector" joint_axis_xyz="${joint_end_effector_axis_xyz}" joint_origin_xyz="${joint_end_effector_origin_xyz}" joint_origin_rpy="${joint_end_effector_origin_rpy}" joint_lower_limit="0" joint_upper_limit="0"/>

File: kinova_description/urdf/kinova_common.xacro (robot description, xacro)
@@ -111,8 +111,8 @@
      </xacro:unless>
   </xacro:macro>
-    <xacro:macro name="kinova_virtual_link" params="link_name">
-        <link name="${link_name}"/>
-    </xacro:macro>
-    <xacro:macro name="kinova_virtual_joint" params="joint_name type parent child joint_axis_xyz joint_origin_xyz joint_origin_rpy joint_lower_limit joint_upper_limit">
+  <xacro:macro name="kinova_virtual_link" params="link_name">
+      <link name="${link_name}"/>
+  </xacro:macro>
+  <xacro:macro name="kinova_virtual_joint" params="joint_name type parent child joint_axis_xyz joint_origin_xyz joint_origin_rpy joint_lower_limit joint_upper_limit">
     <joint name="${joint_name}" type="${type}">
         <parent link="${parent}"/>
@@ -123,43 +123,43 @@
         </xacro:unless>
         <origin xyz="${joint_origin_xyz}" rpy="${joint_origin_rpy}"/>
-     </joint>
-    </xacro:macro>
-    <xacro:macro name="kinova_finger" params="prefix finger_number hand finger_origin_xyz finger_origin_rpy">
-        <xacro:kinova_armlink link_name="${prefix}link_finger_${finger_number}" link_mesh="finger_proximal" mesh_no="57"/>
-        <joint name="${prefix}joint_finger_${finger_number}" type="revolute">
-            <parent link="${hand}"/>
-            <child link="${prefix}link_finger_${finger_number}"/>
-            <axis xyz="0 0 1"/>
-            <origin xyz="${finger_origin_xyz}" rpy="${finger_origin_rpy}"/>
-            <limit lower="0" upper="1.51" effort="2" velocity="1"/>
+    </joint>
+  </xacro:macro>
+  <xacro:macro name="kinova_finger" params="prefix finger_number hand finger_origin_xyz finger_origin_rpy">
+      <xacro:kinova_armlink link_name="${prefix}link_finger_${finger_number}" link_mesh="finger_proximal" mesh_no="57"/>
+      <joint name="${prefix}joint_finger_${finger_number}" type="revolute">
+          <parent link="${hand}"/>
+          <child link="${prefix}link_finger_${finger_number}"/>
+          <axis xyz="0 0 1"/>
+          <origin xyz="${finger_origin_xyz}" rpy="${finger_origin_rpy}"/>
+          <limit lower="0" upper="1.51" effort="2" velocity="1"/>
+      </joint>
+      <transmission name="${prefix}joint_finger_${finger_number}_trans">
+        <type>transmission_interface/SimpleTransmission</type>
+        <joint name="${prefix}joint_finger_${finger_number}">
+          <hardwareInterface>hardware_interface/EffortJointInterface</hardwareInterface>
         </joint>
-		    <transmission name="${prefix}joint_finger_${finger_number}_trans">
-					<type>transmission_interface/SimpleTransmission</type>
-					<joint name="${prefix}joint_finger_${finger_number}">
-					  <hardwareInterface>hardware_interface/EffortJointInterface</hardwareInterface>
-					</joint>
-					<actuator name="${prefix}joint_finger_${finger_number}_actuator">
-					<hardwareInterface>hardware_interface/EffortJointInterface</hardwareInterface>
-					<mechanicalReduction>1</mechanicalReduction>
-					</actuator>
-		    </transmission>
-        <xacro:kinova_armlink link_name="${prefix}link_finger_tip_${finger_number}" link_mesh="finger_distal" mesh_no="58"/>
-        <joint name="${prefix}joint_finger_tip_${finger_number}" type="revolute">
-            <parent link="${prefix}link_finger_${finger_number}"/>
-            <child link="${prefix}link_finger_tip_${finger_number}"/>
-            <axis xyz="0 0 1"/>
-            <origin xyz="0.044 -0.003 0" rpy="0 0 0"/>
-            <limit lower="0" upper="2" effort="2" velocity="1"/>
+        <actuator name="${prefix}joint_finger_${finger_number}_actuator">
+        <hardwareInterface>hardware_interface/EffortJointInterface</hardwareInterface>
+        <mechanicalReduction>1</mechanicalReduction>
+        </actuator>
+      </transmission>
+      <xacro:kinova_armlink link_name="${prefix}link_finger_tip_${finger_number}" link_mesh="finger_distal" mesh_no="58"/>
+      <joint name="${prefix}joint_finger_tip_${finger_number}" type="revolute">
+          <parent link="${prefix}link_finger_${finger_number}"/>
+          <child link="${prefix}link_finger_tip_${finger_number}"/>
+          <axis xyz="0 0 1"/>
+          <origin xyz="0.044 -0.003 0" rpy="0 0 0"/>
+          <limit lower="0" upper="2" effort="2" velocity="1"/>
+      </joint>
+      <transmission name="${prefix}joint_finger_tip_${finger_number}_trans">
+        <type>transmission_interface/SimpleTransmission</type>
+        <joint name="${prefix}joint_finger_tip_${finger_number}">
+          <hardwareInterface>hardware_interface/EffortJointInterface</hardwareInterface>
         </joint>
-        <transmission name="${prefix}joint_finger_tip_${finger_number}_trans">
-					<type>transmission_interface/SimpleTransmission</type>
-					<joint name="${prefix}joint_finger_tip_${finger_number}">
-					  <hardwareInterface>hardware_interface/EffortJointInterface</hardwareInterface>
-					</joint>
-					<actuator name="${prefix}joint_finger_tip_${finger_number}_actuator">
-					<hardwareInterface>hardware_interface/EffortJointInterface</hardwareInterface>
-					<mechanicalReduction>1</mechanicalReduction>
-					</actuator>
-        </transmission>
-    </xacro:macro>
+        <actuator name="${prefix}joint_finger_tip_${finger_number}_actuator">
+        <hardwareInterface>hardware_interface/EffortJointInterface</hardwareInterface>
+        <mechanicalReduction>1</mechanicalReduction>
+        </actuator>
+      </transmission>
+  </xacro:macro>
 </root>
